File: phoenix45_alpha-rounded.kicad_pcb (KiCad board)
At the start: 2 copper layers, 247.7 x 77.5 mm, 114 parts, among them SW1 SW_PUSH, SW2 SW_PUSH, U1 SRV05-4, U3 ATmega32U4-M, X1 Crystal_GND24_Small

Commit message: added avr
Parts:
- added J1: AVR-ISP-6, Connector_IDC:IDC-Header_2x03_P2.54mm_Vertical, F.Cu at (140.0, 34.0)
- moved C6 0.61 mm to (142.7, 44.7)
- moved R1 0.35 mm to (84.4, 43.3)
- moved C5 0.20 mm to (144.2, 41.1)
Connections:
- U3 pad 10: unconnected-(U3-Pad10) -> MOSI
- U3 pad 11: unconnected-(U3-Pad11) -> MISO
- U3 pad 9: unconnected-(U3-Pad9) -> SCK
Routing:
- net MISO: track 0.00 -> 17.2 mm, vias 0 -> 1
- net SCK: track 0.00 -> 15.6 mm, vias 0 -> 1
- net MOSI: track 0.00 -> 14.3 mm, vias 0 -> 1
- net GND: track 71.6 -> 78.6 mm
- net RST: track 77.9 -> 81.6 mm
- net D+: track 112.7 -> 110.1 mm
- net row0: track 262.2 -> 264.8 mm
- net D-: track 114.6 -> 112.3 mm
- net +5V: track 157.8 -> 159.4 mm
- net VCC: track 23.6 -> 22.3 mm
- net col12: track 162.1 -> 160.9 mm
- net Net-(UR4-Pad1): track 13.6 -> 12.6 mm
- net Net-(UR5-Pad1): track 14.1 -> 13.0 mm
- net col8: track 100.1 -> 99.3 mm
- net row2: track 259.3 -> 258.6 mm
