File: phoenix45_alpha.kicad_pcb (KiCad board)
At the start: 2 copper layers, 247.7 x 77.5 mm, 139 parts, among them J1 AVR-ISP-6, SW1 SW_PUSH, SW2 SW_PUSH, SW3 RotaryEncoder_Switch, U1 SRV05-4, U2 ATmega32U4-M, X1 Crystal_GND24_Small

Commit message: minor adjustments
Parts:
- moved R1 3.03 mm to (86.5, 42.1), turned to -90 degrees
- moved C1 1.25 mm to (63.5, 44.1), turned to -90 degrees
- moved F1 0.77 mm to (52.5, 43.1)
Routing:
- net GND: track 63.6 -> 88.3 mm, vias 15 -> 21
- net +5V: track 176.3 -> 181.3 mm
- net col12: track 164.6 -> 161.8 mm
- net col9: track 122.6 -> 125.2 mm
- net col0: track 162.5 -> 164.9 mm
- net Net-(D_SPACE27-Pad2): track 12.9 -> 10.7 mm
- net RST: track 85.9 -> 83.8 mm
- net encA: track 42.4 -> 40.3 mm
- net Net-(D_SPACE43-Pad2): track 10.1 -> 8.35 mm
- net Net-(D_SPACE39-Pad2): track 12.5 -> 10.7 mm
- net Net-(D_SPACE46-Pad2): track 17.2 -> 15.5 mm
- net Net-(D_SPACE44-Pad2): track 10.1 -> 8.35 mm
- net col8: track 103.9 -> 102.2 mm
- net Net-(D_SPACE45-Pad2): track 19.9 -> 19.1 mm
- net SDA: track 17.6 -> 18.4 mm
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